Commit message: Stepper motor changes required following the implementation of dynamixel_hardware_interface (actionLib)

File: model/urdf/maggie.urdf (robot description, URDF)
Before this commit: robot pi_robot, 18 links, 17 joints
Links:
- added link r_gripper_l_finger_link, mass 0.17126; collision mesh filename=package://pr2_description/meshes/gripper_v0/l_finger.stl; visual mesh filename=package://pr2_description/meshes/gripper_v0/l_finger.dae
- added link r_gripper_l_finger_tip_frame
- added link r_gripper_l_finger_tip_link, mass 0.04419; collision mesh filename=package://pr2_description/meshes/gripper_v0/l_finger_tip.stl; visual mesh filename=package://pr2_description/meshes/gripper_v0/l_finger_tip.dae
- added link r_gripper_led_frame
- added link r_gripper_motor_accelerometer_link, mass 0.001; collision box size=0.001 0.001 0.001; visual box size=0.001 0.001 0.001
- added link r_gripper_motor_screw_link, mass 0.01
- added link r_gripper_motor_slider_link, mass 0.01
- added link r_gripper_palm_link, mass 0.58007; collision mesh filename=package://pr2_description/meshes/gripper_v0/gripper_palm.stl; visual mesh filename=package://pr2_description/meshes/gripper_v0/gripper_palm.dae
- added link r_gripper_r_finger_link, mass 0.17389; collision mesh filename=package://pr2_description/meshes/gripper_v0/l_finger.stl; visual mesh filename=package://pr2_description/meshes/gripper_v0/l_finger.dae
- added link r_gripper_r_finger_tip_link, mass 0.04419; collision mesh filename=package://pr2_description/meshes/gripper_v0/l_finger_tip.stl; visual mesh filename=package://pr2_description/meshes/gripper_v0/l_finger_tip.dae
- added link r_gripper_tool_frame
- added link wrist_tilt_link; collision box size=0.03 0.003 0.03; visual box size=0.03 0.003 0.03
Joints:
- added joint r_gripper_joint: type prismatic, parent r_gripper_r_finger_tip_link, child r_gripper_l_finger_tip_frame, axis 0 1 0, limit lower=0.0 upper=0.09 effort=1000.0 velocity=0.2
- added joint r_gripper_l_finger_joint: type revolute, parent r_gripper_palm_link, child r_gripper_l_finger_link, origin xyz=0.07691 0.01 0 rpy=0 0 0, axis 0 0 1, limit lower=0.0 upper=0.548 effort=1000.0 velocity=0.5
- added joint r_gripper_l_finger_tip_joint: type revolute, parent r_gripper_l_finger_link, child r_gripper_l_finger_tip_link, origin xyz=0.09137 0.00495 0 rpy=0 0 0, axis 0 0 -1, limit lower=0.0 upper=0.548 effort=1000.0 velocity=0.5, mimic joint=r_gripper_l_finger_joint multiplier=1 offset=0
- added joint r_gripper_led_joint: type fixed, parent r_gripper_palm_link, child r_gripper_led_frame, origin xyz=0.0513 0.0 .0244
- added joint r_gripper_motor_accelerometer_joint: type fixed, parent r_gripper_palm_link, child r_gripper_motor_accelerometer_link, origin xyz=0 0 0 rpy=0 0 0
- added joint r_gripper_motor_screw_joint: type continuous, parent r_gripper_motor_slider_link, child r_gripper_motor_screw_link, origin xyz=0.0 0 0 rpy=0 0 0, axis 0 1 0
- added joint r_gripper_motor_slider_joint: type prismatic, parent r_gripper_palm_link, child r_gripper_motor_slider_link, origin xyz=0.16828 0 0 rpy=0 0 0, axis 1 0 0, limit lower=-0.1 upper=0.1 effort=1000.0 velocity=0.2
- added joint r_gripper_palm_joint: type fixed, parent wrist_tilt_link, child r_gripper_palm_link, origin xyz=0 0 0 rpy=0 0 0
- added joint r_gripper_r_finger_joint: type revolute, parent r_gripper_palm_link, child r_gripper_r_finger_link, origin xyz=0.07691 -0.01 0 rpy=0 0 0, axis 0 0 -1, limit lower=0.0 upper=0.548 effort=1000.0 velocity=0.5, mimic joint=r_gripper_l_finger_joint multiplier=1 offset=0
- added joint r_gripper_r_finger_tip_joint: type revolute, parent r_gripper_r_finger_link, child r_gripper_r_finger_tip_link, origin xyz=0.09137 -0.00495 0 rpy=0 0 0, axis 0 0 1, limit lower=0.0 upper=0.548 effort=1000.0 velocity=0.5, mimic joint=r_gripper_l_finger_joint multiplier=1 offset=0
- added joint r_gripper_tool_joint: type fixed, parent r_gripper_palm_link, child r_gripper_tool_frame, origin xyz=0.18 0 0 rpy=0 0 0
- added joint wrist_tilt_joint: type revolute, parent forearm_link, child wrist_tilt_link, origin xyz=0.255 0 0 rpy=0 0 0, axis 0 1 0, limit lower=-1.0 upper=1.0 effort=1.0 velocity=1.0

File: model/urdf/maggie.xacro (robot description, xacro)
@@ -5,8 +5,7 @@
        xmlns:interface="http://playerstage.sourceforge.net/gazebo/xmlschema/#interface"
        xmlns:xacro="http://ros.org/wiki/xacro"
-	   name="pi_robot">
-	<!--
-	<include filename="$(find pi_robot_description)/urdf/sensors/hokuyo_laser_gazebo.xacro" />
-	-->
+	   name="maggie">
+	<include filename="$(find pr2_description)/urdf/materials.urdf.xacro" />
+	<include filename="$(find pr2_description)/urdf/gripper_v0/gripper.urdf.xacro" />
 	<xacro:macro name="white">
 		<material name="white">
@@ -123,6 +122,22 @@
 	</xacro:my_box>
 	<xacro:my_cylinder name="forearm_link" l="0.27" r="0.025" xyz="0.135 0 0" rpy="0 1.57 0" mass="0.5" material="Gazebo/WhiteEmissive">
-		<xacro:red1 />
-	</xacro:my_cylinder>
+		<xacro:grey1 />
+	</xacro:my_cylinder>
+	<xacro:my_box name="wrist_tilt_link" lwh="0.03 0.003 0.03" xyz="0.015 0 0" rpy="0 0 0" mass="0.5" material="Gazebo/WhiteEmissive">
+		<xacro:blue1 />
+	</xacro:my_box>
+	<xacro:pr2_gripper_v0 reflect="-1.0" side="r" parent="wrist_tilt_link"
+               screw_reduction="${4.0/1000.0}"
+               gear_ratio="${(729.0/25.0)*(22.0/16.0)}"
+               theta0="${3.6029*M_PI/180.0}"
+               phi0="${29.7089*M_PI/180.0}"
+               t0="${-0.1914/1000.0}"
+               L0="${37.5528/1000.0}"
+               h="${0.0/1000.0}"
+               a="${68.3698/1000.0}"
+               b="${43.3849/1000.0}"
+               r="${91.5/1000.0}" >
+	<origin xyz="0 0 0" rpy="0 0 0" />
+      </xacro:pr2_gripper_v0>
 	<!-- head links -->
 	<xacro:my_cylinder name="lower_neck_link" l="0.16" r="0.025" xyz="0 0 0" rpy="0 0 0" mass="0.05" material="Gazebo/WhiteEmissive">
@@ -208,4 +223,11 @@
 	</joint>
 	<!-- arm joints -->
+	<joint name="wrist_tilt_joint" type="revolute">
+	  <parent link="forearm_link" />
+	  <child link="wrist_tilt_link" />
+	  <axis xyz="0 1 0"/>
+	  <origin xyz="0.255 0 0" rpy="0 0 0" />
+	  <limit lower="-1.0" upper="1.0" effort="1.0" velocity="1.0" />
+	</joint>
 	<joint name="forearm_roll_joint" type="revolute">
 	  <parent link="elbow_tilt_link" />
