Commit message: model and IK changes

File: maggie_model/urdf/maggie.urdf (robot description, URDF)
Before this commit: robot maggie, 30 links, 29 joints
Links:
- removed link r_gripper_l_finger_link
- removed link r_gripper_l_finger_tip_frame
- removed link r_gripper_l_finger_tip_link
- removed link r_gripper_led_frame
- removed link r_gripper_motor_accelerometer_link
- removed link r_gripper_motor_screw_link
- removed link r_gripper_motor_slider_link
- removed link r_gripper_palm_link
- removed link r_gripper_r_finger_link
- removed link r_gripper_r_finger_tip_link
- removed link r_gripper_tool_frame
- added link hand_link; collision box size=0.01 0.01 0.005; visual box size=0.01 0.01 0.005
- added link wrist_roll_link; collision box size=0.02 0.003 0.03; visual box size=0.02 0.003 0.03
- link elbow_tilt_link: geometry collision box size=0.1 0.003 0.03; visual box size=0.1 0.003 0.03
- link forearm_link: geometry collision cylinder length=0.151 radius=0.025; visual cylinder length=0.151 radius=0.025
- link shoulder_pan_support_link: geometry collision box size=0.08 0.04 0.005; visual box size=0.08 0.04 0.005
- link shoulder_tilt_link: geometry collision box size=0.15 0.003 0.02; visual box size=0.15 0.003 0.02
- link shoulder_tilt_support_link: geometry collision box size=0.07 0.003 0.06; visual box size=0.07 0.003 0.06
- link upper_arm_link: geometry collision cylinder length=0.08 radius=0.025; visual cylinder length=0.08 radius=0.025
- link wrist_tilt_link: geometry collision box size=0.0355 0.003 0.03; visual box size=0.0355 0.003 0.03
Joints:
- removed joint r_gripper_joint
- removed joint r_gripper_l_finger_joint
- removed joint r_gripper_l_finger_tip_joint
- removed joint r_gripper_led_joint
- removed joint r_gripper_motor_accelerometer_joint
- removed joint r_gripper_motor_screw_joint
- removed joint r_gripper_motor_slider_joint
- removed joint r_gripper_palm_joint
- removed joint r_gripper_r_finger_joint
- removed joint r_gripper_r_finger_tip_joint
- removed joint r_gripper_tool_joint
- added joint hand_joint: type fixed, parent wrist_roll_link, child hand_link, origin xyz=0.02 0 0 rpy=0 0 0
- added joint wrist_roll_joint: type revolute, parent wrist_tilt_link, child wrist_roll_link, origin xyz=0.0351 0 0 rpy=0 0 0, axis 1 0 0, limit lower=-2.61 upper=2.61 effort=1.0 velocity=1.0
- joint elbow_tilt_joint: limit lower=-1.0 upper=1.0 effort=1.0 velocity=1.0 -> lower=-2.61 upper=2.61 effort=1.0 velocity=1.0; origin xyz=0.27 0 0 rpy=0 0 0 -> xyz=0.07 0 0 rpy=0 -1.57 0
- joint forearm_roll_joint: axis 0.135 0 0 -> 1 0 0; limit lower=-1.0 upper=1.0 effort=1.0 velocity=1.0 -> lower=-2.61 upper=2.61 effort=1.0 velocity=1.0; origin xyz=0 0 0 rpy=0 0 0 -> xyz=0.1 0 0 rpy=0 0 0
- joint shoulder_pan_joint: limit lower=-1.0 upper=1.0 effort=1.0 velocity=1.0 -> lower=-1.57 upper=1.57 effort=1.0 velocity=1.0
- joint shoulder_pan_support_joint: origin xyz=0.0325 -0.14 0.173 rpy=0 0 0 -> xyz=0.0425 -0.14 0.173 rpy=0 0 0
- joint shoulder_tilt_joint: limit lower=-1.0 upper=1.0 effort=1.0 velocity=1.0 -> lower=-1.57 upper=1.57 effort=1.0 velocity=1.0; origin xyz=0 0 -0.015 rpy=0 0 0 -> xyz=0.03 -0.05 0 rpy=0 0 0
- joint shoulder_tilt_support_joint: origin xyz=0.0175 0.0 0 rpy=0 0 0 -> xyz=0.04 0.05 0.05 rpy=0 0 0
- joint upper_arm_roll_joint: axis 0.135 0 0 -> 1 0 0; limit lower=-1.0 upper=1.0 effort=1.0 velocity=1.0 -> lower=-2.61 upper=2.61 effort=1.0 velocity=1.0; origin xyz=0 0 0 rpy=0 0 0 -> xyz=0.1 0 0 rpy=0 0 0
- joint wrist_tilt_joint: limit lower=-1.0 upper=1.0 effort=1.0 velocity=1.0 -> lower=-1.57 upper=1.57 effort=1.0 velocity=1.0; origin xyz=0.255 0 0 rpy=0 0 0 -> xyz=0.151 0 0 rpy=0 0 0

File: maggie_model/urdf/maggie.xacro (robot description, xacro)
@@ -112,9 +112,9 @@
 		<xacro:blue1 />
 	</xacro:my_box>
-	<xacro:my_box name="shoulder_tilt_link" lwh="0.1 0.003 0.02" xyz="0.05 0 0" rpy="0 0 0" mass="0.5" material="Gazebo/WhiteEmissive">
-		<xacro:green1 />
-	</xacro:my_box>
-	<xacro:my_cylinder name="upper_arm_link" l="0.224" r="0.025" xyz="0.135 0 0" rpy="0 1.57 0" mass="0.5" material="Gazebo/WhiteEmissive">
+	<xacro:my_box name="shoulder_tilt_link" lwh="0.15 0.003 0.02" xyz="0.075 0 0" rpy="0 0 0" mass="0.5" material="Gazebo/WhiteEmissive">
 		<xacro:red1 />
+	</xacro:my_box>
+	<xacro:my_cylinder name="upper_arm_link" l="0.08" r="0.025" xyz="0.035 0 0" rpy="0 1.57 0" mass="0.5" material="Gazebo/WhiteEmissive">
+		<xacro:blue1 />
 	</xacro:my_cylinder>
 	<xacro:my_box name="elbow_tilt_link" lwh="0.1 0.003 0.03" xyz="0.05 0 0" rpy="0 0 0" mass="0.5" material="Gazebo/WhiteEmissive">
@@ -124,11 +124,20 @@
 		<xacro:grey1 />
 	</xacro:my_cylinder>
-	<xacro:my_box name="wrist_tilt_link" lwh="0.03 0.003 0.03" xyz="0.015 0 0" rpy="0 0 0" mass="0.5" material="Gazebo/WhiteEmissive">
+	<xacro:my_box name="wrist_tilt_link" lwh="0.0355 0.003 0.03" xyz="0.01775 0 0" rpy="0 0 0" mass="0.5" material="Gazebo/WhiteEmissive">
 		<xacro:blue1 />
 	</xacro:my_box>
-	<xacro:my_box name="wrist_roll_link" lwh="0.071 0.003 0.03" xyz="0.03 0 0" rpy="0 0 0" mass="0.5" material="Gazebo/WhiteEmissive">
+	<xacro:my_box name="wrist_roll_link" lwh="0.02 0.003 0.03" xyz="0.01 0 0" rpy="0 0 0" mass="0.5" material="Gazebo/WhiteEmissive">
 		<xacro:red1 />
 	</xacro:my_box>
-<!--	<xacro:pr2_gripper_v0 reflect="-1.0" side="r" parent="wrist_roll_link"
+	<xacro:my_box name="hand_link" lwh="0.01 0.01 0.005" xyz="0.005 0 0" rpy="0 0 0" mass="0.001" material="Gazebo/WhiteEmissive">
+	  <xacro:green1 />
+	</xacro:my_box>
+<!--	<xacro:my_box name="hand_link" lwh="0.03 0.01 0.064" xyz="0 0 -0.032" rpy="0 0 0" mass="0.1" material="Gazebo/WhiteEmissive">
+	  <xacro:grey1 />
+	</xacro:my_box>-->
+<!--	<xacro:my_box name="finger_link" lwh="0.01 0.01 0.005" xyz="0 0 0" rpy="0 0 0" mass="0.001" material="Gazebo/WhiteEmissive">
+	  <xacro:green1 />
+	</xacro:my_box>-->
+	<!--xacro:pr2_gripper_v0 reflect="-1.0" side="r" parent="wrist_roll_link"
                screw_reduction="${4.0/1000.0}"
                gear_ratio="${(729.0/25.0)*(22.0/16.0)}"
@@ -142,5 +151,5 @@
                r="${91.5/1000.0}" >
 	<origin xyz="0 0 0" rpy="0 0 0" />
-      </xacro:pr2_gripper_v0>-->
+      </xacro:pr2_gripper_v0-->
 	<!-- head links -->
 	<xacro:my_cylinder name="lower_neck_link" l="0.16" r="0.025" xyz="0 0 0" rpy="0 0 0" mass="0.05" material="Gazebo/WhiteEmissive">
@@ -226,17 +235,27 @@
 	</joint>
 	<!-- arm joints -->
+<!--        <joint name="finger_joint" type="fixed">
+	  <parent link="hand_link" />
+	  <child link="finger_link" />
+	  <origin xyz="0 0 -0.064" rpy="0 0 0" />
+        </joint>-->
+	<joint name="hand_joint" type="fixed">
+	  <parent link="wrist_roll_link" />
+	  <child link="hand_link" />
+	  <origin xyz="0.02 0 0" rpy="0 0 0" />
+        </joint>
 	<joint name="wrist_roll_joint" type="revolute">
 	  <parent link="wrist_tilt_link" />
 	  <child link="wrist_roll_link" />
 	  <axis xyz="1 0 0"/>
-	  <origin xyz="0.035 0 0" rpy="0 0 0" />
-	  <limit lower="-1.0" upper="1.0" effort="1.0" velocity="1.0" />
+	  <origin xyz="0.0351 0 0" rpy="0 0 0" />
+	  <limit lower="-2.61" upper="2.61" effort="1.0" velocity="1.0" />
 	</joint>
 	<joint name="wrist_tilt_joint" type="revolute">
 	  <parent link="forearm_link" />
 	  <child link="wrist_tilt_link" />
-	  <axis xyz="0 -1 0"/>
+	  <axis xyz="0 1 0"/>
 	  <origin xyz="0.151 0 0" rpy="0 0 0" />
-	  <limit lower="-1.0" upper="1.0" effort="1.0" velocity="1.0" />
+	  <limit lower="-1.57" upper="1.57" effort="1.0" velocity="1.0" />
 	</joint>
 	<joint name="forearm_roll_joint" type="revolute">
@@ -245,5 +264,5 @@
 	  <axis xyz="1 0 0"/>
 	  <origin xyz="0.1 0 0" rpy="0 0 0" />
-	  <limit lower="-1.0" upper="1.0" effort="1.0" velocity="1.0" />
+	  <limit lower="-2.61" upper="2.61" effort="1.0" velocity="1.0" />
 	</joint>
 	<joint name="elbow_tilt_joint" type="revolute">
@@ -251,6 +270,6 @@
 	  <child link="elbow_tilt_link" />
 	  <axis xyz="0 1 0"/>
-	  <origin xyz="0.27 0 0" rpy="0 -1.57 0" />
-	  <limit lower="-1.0" upper="1.0" effort="1.0" velocity="1.0" />
+	  <origin xyz="0.07 0 0" rpy="0 -1.57 0" />
+	  <limit lower="-2.61" upper="2.61" effort="1.0" velocity="1.0" />
 	</joint>
 	<joint name="upper_arm_roll_joint" type="revolute">
@@ -259,5 +278,5 @@
 	  <axis xyz="1 0 0"/>
 	  <origin xyz="0.1 0 0" rpy="0 0 0" />
-	  <limit lower="-1.0" upper="1.0" effort="1.0" velocity="1.0" />
+	  <limit lower="-2.61" upper="2.61" effort="1.0" velocity="1.0" />
 	</joint>
 	<joint name="shoulder_tilt_joint" type="revolute">
@@ -265,6 +284,6 @@
 	  <child link="shoulder_tilt_link" />
 	  <axis xyz="0 1 0"/>
-	  <origin xyz="0.035 -0.05 0" rpy="0 0 0" />
-	  <limit lower="-1.0" upper="1.0" effort="1.0" velocity="1.0" />
+	  <origin xyz="0.03 -0.05 0" rpy="0 0 0" />
+	  <limit lower="-1.57" upper="1.57" effort="1.0" velocity="1.0" />
 	</joint>
 	<joint name="shoulder_tilt_support_joint" type="fixed">
@@ -278,5 +297,5 @@
 	  <axis xyz="0.0 0 1"/>
 	  <origin xyz="0.03 0 0" rpy="0 0 0" />
-	  <limit lower="-1.0" upper="1.0" effort="1.0" velocity="1.0" />
+	  <limit lower="-1.57" upper="1.57" effort="1.0" velocity="1.0" />
 	</joint>
 	<joint name="shoulder_pan_support_joint" type="fixed">

Commit message: Further accuracy tweaks to the .xacro file

File: maggie_model/urdf/maggie.urdf (robot description, URDF)
Before this commit: robot maggie, 21 links, 20 joints
Links:
- link shoulder_tilt_link: geometry collision box size=0.1 0.003 0.02; visual box size=0.1 0.003 0.02
- link shoulder_tilt_support_link: geometry collision box size=0.068 0.003 0.06; visual box size=0.068 0.003 0.06
- link torso_link: geometry collision box size=0.005 0.4 0.752; visual box size=0.005 0.4 0.752
- link upper_arm_link: geometry collision cylinder length=0.13 radius=0.025; visual cylinder length=0.13 radius=0.025
- link wrist_roll_link: geometry collision box size=0.035 0.003 0.03; visual box size=0.035 0.003 0.03
- link wrist_tilt_link: geometry collision box size=0.036 0.003 0.03; visual box size=0.036 0.003 0.03
Joints:
- joint elbow_tilt_joint: origin xyz=0.07 0 0 rpy=0 -1.57 0 -> xyz=0.129 0 0 rpy=0 -1.57 0
- joint forearm_roll_joint: origin xyz=0.1 0 0 rpy=0 0 0 -> xyz=0.1 0 0.012 rpy=0 0 0
- joint hand_joint: origin xyz=0.02 0 0 rpy=0 0 0 -> xyz=0.0351 0 0 rpy=0 0 0
- joint shoulder_pan_joint: origin xyz=0.03 0 0 rpy=0 0 0 -> xyz=0.04 0 0 rpy=0 0 0
- joint shoulder_pan_support_joint: origin xyz=0.0425 -0.14 0.173 rpy=0 0 0 -> xyz=0.0425 -0.14 0.175 rpy=0 0 0
- joint shoulder_tilt_joint: origin xyz=0.03 -0.05 0 rpy=0 0 0 -> xyz=0.034 -0.05 0 rpy=0 0 0
- joint shoulder_tilt_support_joint: origin xyz=0.04 0.05 0.05 rpy=0 0 0 -> xyz=0.034 0.05 0.05 rpy=0 0 0
- joint torso_joint: origin xyz=0 0 0.375 rpy=0 0 0 -> xyz=0 0 0.376 rpy=0 0 0
- joint upper_arm_roll_joint: origin xyz=0.1 0 0 rpy=0 0 0 -> xyz=0.1 0 0.025 rpy=0 0 0
- joint wrist_tilt_joint: origin xyz=0.151 0 0 rpy=0 0 0 -> xyz=0.152 0 0.002 rpy=0 0 0

File: maggie_model/urdf/maggie.xacro (robot description, xacro)
@@ -100,5 +100,5 @@
 		<xacro:white />
 	</xacro:my_box>
- 	<xacro:my_box name="torso_link" lwh="0.005 0.4 0.75" xyz="0 0 0" rpy="0 0 0" mass="0.5" material="Gazebo/WhiteEmissive">
+ 	<xacro:my_box name="torso_link" lwh="0.005 0.4 0.752" xyz="0 0 0" rpy="0 0 0" mass="0.5" material="Gazebo/WhiteEmissive">
 		<xacro:grey1 />
 	</xacro:my_box>
@@ -109,11 +109,11 @@
 		<xacro:green1 />
 	</xacro:my_cylinder>
-	<xacro:my_box name="shoulder_tilt_support_link" lwh="0.07 0.003 0.06" xyz="0 0 0" rpy="0 0 0" mass="0.5" material="Gazebo/WhiteEmissive">
+	<xacro:my_box name="shoulder_tilt_support_link" lwh="0.068 0.003 0.06" xyz="0 0 0" rpy="0 0 0" mass="0.5" material="Gazebo/WhiteEmissive">
 		<xacro:blue1 />
 	</xacro:my_box>
-	<xacro:my_box name="shoulder_tilt_link" lwh="0.15 0.003 0.02" xyz="0.075 0 0" rpy="0 0 0" mass="0.5" material="Gazebo/WhiteEmissive">
+	<xacro:my_box name="shoulder_tilt_link" lwh="0.1 0.003 0.02" xyz="0.05 0 0" rpy="0 0 0" mass="0.5" material="Gazebo/WhiteEmissive">
 		<xacro:red1 />
 	</xacro:my_box>
-	<xacro:my_cylinder name="upper_arm_link" l="0.08" r="0.025" xyz="0.035 0 0" rpy="0 1.57 0" mass="0.5" material="Gazebo/WhiteEmissive">
+	<xacro:my_cylinder name="upper_arm_link" l="0.13" r="0.025" xyz="0.065 0 0" rpy="0 1.57 0" mass="0.5" material="Gazebo/WhiteEmissive">
 		<xacro:blue1 />
 	</xacro:my_cylinder>
@@ -124,8 +124,8 @@
 		<xacro:grey1 />
 	</xacro:my_cylinder>
-	<xacro:my_box name="wrist_tilt_link" lwh="0.0355 0.003 0.03" xyz="0.01775 0 0" rpy="0 0 0" mass="0.5" material="Gazebo/WhiteEmissive">
+	<xacro:my_box name="wrist_tilt_link" lwh="0.036 0.003 0.03" xyz="0.018 0 0" rpy="0 0 0" mass="0.5" material="Gazebo/WhiteEmissive">
 		<xacro:blue1 />
 	</xacro:my_box>
-	<xacro:my_box name="wrist_roll_link" lwh="0.02 0.003 0.03" xyz="0.01 0 0" rpy="0 0 0" mass="0.5" material="Gazebo/WhiteEmissive">
+	<xacro:my_box name="wrist_roll_link" lwh="0.035 0.003 0.03" xyz="0.0175 0 0" rpy="0 0 0" mass="0.5" material="Gazebo/WhiteEmissive">
 		<xacro:red1 />
 	</xacro:my_box>
@@ -243,5 +243,5 @@
 	  <parent link="wrist_roll_link" />
 	  <child link="hand_link" />
-	  <origin xyz="0.02 0 0" rpy="0 0 0" />
+	  <origin xyz="0.0351 0 0" rpy="0 0 0" />
         </joint>
 	<joint name="wrist_roll_joint" type="revolute">
@@ -256,5 +256,5 @@
 	  <child link="wrist_tilt_link" />
 	  <axis xyz="0 1 0"/>
-	  <origin xyz="0.151 0 0" rpy="0 0 0" />
+	  <origin xyz="0.152 0 0.002" rpy="0 0 0" />
 	  <limit lower="-1.57" upper="1.57" effort="1.0" velocity="1.0" />
 	</joint>
@@ -263,5 +263,5 @@
 	  <child link="forearm_link" />
 	  <axis xyz="1 0 0"/>
-	  <origin xyz="0.1 0 0" rpy="0 0 0" />
+	  <origin xyz="0.1 0 0.012" rpy="0 0 0" />
 	  <limit lower="-2.61" upper="2.61" effort="1.0" velocity="1.0" />
 	</joint>
@@ -270,5 +270,5 @@
 	  <child link="elbow_tilt_link" />
 	  <axis xyz="0 1 0"/>
-	  <origin xyz="0.07 0 0" rpy="0 -1.57 0" />
+	  <origin xyz="0.129 0 0" rpy="0 -1.57 0" />
 	  <limit lower="-2.61" upper="2.61" effort="1.0" velocity="1.0" />
 	</joint>
@@ -277,5 +277,5 @@
 	  <child link="upper_arm_link" />
 	  <axis xyz="1 0 0"/>
-	  <origin xyz="0.1 0 0" rpy="0 0 0" />
+	  <origin xyz="0.1 0 0.025" rpy="0 0 0" />
 	  <limit lower="-2.61" upper="2.61" effort="1.0" velocity="1.0" />
 	</joint>
@@ -284,5 +284,5 @@
 	  <child link="shoulder_tilt_link" />
 	  <axis xyz="0 1 0"/>
-	  <origin xyz="0.03 -0.05 0" rpy="0 0 0" />
+	  <origin xyz="0.034 -0.05 0" rpy="0 0 0" />
 	  <limit lower="-1.57" upper="1.57" effort="1.0" velocity="1.0" />
 	</joint>
@@ -290,5 +290,5 @@
 	  <parent link="shoulder_pan_link" />
 	  <child link="shoulder_tilt_support_link" />
-	  <origin xyz="0.04 0.05 0.05" rpy="0 0 0" />
+	  <origin xyz="0.034 0.05 0.05" rpy="0 0 0" />
 	</joint>
 	<joint name="shoulder_pan_joint" type="revolute">
@@ -296,5 +296,5 @@
 	  <child link="shoulder_pan_link" />
 	  <axis xyz="0.0 0 1"/>
-	  <origin xyz="0.03 0 0" rpy="0 0 0" />
+	  <origin xyz="0.04 0 0" rpy="0 0 0" />
 	  <limit lower="-1.57" upper="1.57" effort="1.0" velocity="1.0" />
 	</joint>
@@ -302,10 +302,10 @@
 	  <parent link="torso_link" />
 	  <child link="shoulder_pan_support_link" />
-	  <origin xyz="0.0425 -0.14 0.173" rpy="0 0 0" />
+	  <origin xyz="0.0425 -0.14 0.175" rpy="0 0 0" />
 	</joint>
 	<joint name="torso_joint" type="fixed">
 	  <parent link="base_link" />
 	  <child link="torso_link" />
-	  <origin xyz="0 0 0.375" rpy="0 0 0" />
+	  <origin xyz="0 0 0.376" rpy="0 0 0" />
 	</joint>
 	<gazebo reference="maggie">

Commit message: Further changes to maggie.xacrox

File: maggie_model/urdf/maggie.urdf (robot description, URDF)
Before this commit: robot maggie, 21 links, 20 joints
Links:
- removed link upper_neck_link
- added link head_pan_servo_link; collision box size=0.05 0.035 0.044; visual box size=0.05 0.035 0.044
- link head_pan_link: geometry collision box size=0.05 0.035 0.044; visual box size=0.05 0.035 0.044
- link head_tilt_link: geometry collision box size=0.03 0.038 0.030; visual box size=0.03 0.038 0.030
Joints:
- joint head_base_joint: origin xyz=0 0 0.016 rpy=0 0 0 -> xyz=0 0 0.022 rpy=0 0 0
- joint head_joint: origin xyz=0 0 0.0235 rpy=0 0 0 -> xyz=0 0 0.012 rpy=0 0 0
- joint head_pan_joint: child head_tilt_link -> head_pan_link; origin xyz=0.01 0 0.048 rpy=0 0 0 -> xyz=0 0 0.044 rpy=0 0 0; parent head_pan_link -> head_pan_servo_link
- joint head_pan_servo_joint: child head_pan_link -> head_pan_servo_link; origin xyz=0.02 0 0.1 rpy=0 0 0 -> xyz=0.029 0 0.16 rpy=0 0 0
- joint head_tilt_joint: child upper_neck_link -> head_tilt_link; origin xyz=0 0 0.013 rpy=0 0 0 -> xyz=0 0 0.044 rpy=0 0 0; parent head_tilt_link -> head_pan_link
- joint lower_neck_joint: origin xyz=-0.0275 0 0.455 rpy=0 0 0 -> xyz=-0.0275 0 0.376 rpy=0 0 0
- joint upper_neck_joint: origin xyz=0 0 0.040 rpy=0 0 0 -> xyz=0 0 0.030 rpy=0 0 0; parent upper_neck_link -> head_tilt_link

File: maggie_model/urdf/maggie.xacro (robot description, xacro)
@@ -153,29 +153,32 @@
       </xacro:pr2_gripper_v0-->
 	<!-- head links -->
-	<xacro:my_cylinder name="lower_neck_link" l="0.16" r="0.025" xyz="0 0 0" rpy="0 0 0" mass="0.05" material="Gazebo/WhiteEmissive">
-		<xacro:grey1 />
-	</xacro:my_cylinder>
-	<xacro:my_box name="upper_neck_link" lwh="0.028 0.048 0.037" xyz="0 0 0.01" rpy="0 0 0" mass="0.05" material="Gazebo/WhiteEmissive">
+	<xacro:my_cylinder name="lower_neck_link" l="0.16" r="0.025" xyz="0 0 0.079" rpy="0 0 0" mass="0.05" material="Gazebo/WhiteEmissive">
+		<xacro:grey1 />
+	</xacro:my_cylinder>
+<!--	<xacro:my_box name="upper_neck_link" lwh="0.026 0.048 0.026" xyz="0 0 0.013" rpy="0 0 0" mass="0.05" material="Gazebo/WhiteEmissive">
 		<xacro:bracket_color />
-	</xacro:my_box>
-	<xacro:my_box name="head_pan_link" lwh="0.05 0.035 0.04" xyz="0 0 0" rpy="0 0 0" mass="0.055" material="Gazebo/FlatBlack">
+	</xacro:my_box>-->
+	<xacro:my_box name="head_pan_servo_link" lwh="0.05 0.035 0.044" xyz="-0.01 0 0.022" rpy="0 0 0" mass="0.055" material="Gazebo/FlatBlack">
 		<xacro:ax12_color />
 	</xacro:my_box>
-	<xacro:my_box name="head_tilt_link" lwh="0.03 0.038 0.057" xyz="0 0 0" rpy="0 0 0" mass="0.055" material="Gazebo/FlatBlack">
+	<xacro:my_box name="head_pan_link" lwh="0.05 0.035 0.044" xyz="-0.01 0 0.022" rpy="0 0 0" mass="0.055" material="Gazebo/FlatBlack">
 		<xacro:ax12_color />
 	</xacro:my_box>
-	<xacro:my_box name="head_base_link" lwh="0.06 0.08 0.022" xyz="0 0 00" rpy="0 0 0" mass="0.1" material="Gazebo/FlatBlack">
+	<xacro:my_box name="head_tilt_link" lwh="0.03 0.038 0.030" xyz="0 0 0.015" rpy="0 0 0" mass="0.055" material="Gazebo/FlatBlack">
+		<xacro:ax12_color />
+	</xacro:my_box>
+	<xacro:my_box name="head_base_link" lwh="0.06 0.08 0.022" xyz="0 0 0.011" rpy="0 0 0" mass="0.1" material="Gazebo/FlatBlack">
 		<xacro:black />
 	</xacro:my_box>
-	<xacro:my_cylinder name="head_post_link" l="0.012" r="0.005" xyz="0 0 00" rpy="0 0 0" mass="0.1" material="Gazebo/WhiteEmissive">
-		<xacro:grey1 />
-	</xacro:my_cylinder>
-	<xacro:my_box name="head_link" lwh="0.06 0.26 0.035" xyz="0 0 00" rpy="0 0 0" mass="0.8" material="Gazebo/FlatBlack">
+	<xacro:my_cylinder name="head_post_link" l="0.012" r="0.005" xyz="0 0 0.006" rpy="0 0 0" mass="0.1" material="Gazebo/WhiteEmissive">
+		<xacro:grey1 />
+	</xacro:my_cylinder>
+	<xacro:my_box name="head_link" lwh="0.06 0.26 0.035" xyz="0 0 0.0175" rpy="0 0 0" mass="0.8" material="Gazebo/FlatBlack">
 		<xacro:black />
 	</xacro:my_box>
-	<xacro:my_cylinder name="left_eye_link" l="0.01" r="0.01" xyz="0 0 00" rpy="0 0 0" mass="0.001" material="Gazebo/WhiteEmissive">
-		<xacro:grey1 />
-	</xacro:my_cylinder>
-	<xacro:my_cylinder name="right_eye_link" l="0.01" r="0.01" xyz="0 0 00" rpy="0 0 0" mass="0.001" material="Gazebo/WhiteEmissive">
+	<xacro:my_cylinder name="left_eye_link" l="0.01" r="0.01" xyz="0 0 0" rpy="0 0 0" mass="0.001" material="Gazebo/WhiteEmissive">
+		<xacro:grey1 />
+	</xacro:my_cylinder>
+	<xacro:my_cylinder name="right_eye_link" l="0.01" r="0.01" xyz="0 0 0" rpy="0 0 0" mass="0.001" material="Gazebo/WhiteEmissive">
 		<xacro:grey1 />
 	</xacro:my_cylinder>
@@ -186,58 +189,53 @@
     	<parent link="torso_link" />
     	<child link="lower_neck_link" />
-    	<origin xyz="-0.0275 0 0.455" rpy="0 0 0" />
+    	<origin xyz="-0.0275 0 0.376" rpy="0 0 0" />
 	</joint>
 	<joint name="head_pan_servo_joint" type="fixed">
     	<parent link="lower_neck_link" />
+    	<child link="head_pan_servo_link" />
+    	<origin xyz="0.029 0 0.16" rpy="0 0 0" />
+	</joint>
+	<joint name="head_pan_joint" type="revolute">
+    	<parent link="head_pan_servo_link" />
     	<child link="head_pan_link" />
-    	<origin xyz="0.02 0 0.1" rpy="0 0 0" />
-	</joint>
-	<joint name="head_pan_joint" type="revolute">
-    	<parent link="head_pan_link" />
-    	<child link="head_tilt_link" />
-    	<origin xyz="0.01 0 0.048" rpy="0 0 0" />
+    	<origin xyz="0 0 0.044" rpy="0 0 0" />
     	<axis xyz="0 0 1" />
     	<limit lower="-3.1416" upper="3.1416" effort="10" velocity="3" />
       	<dynamics damping="0.0"/>
 	</joint>
- 	<joint name="head_tilt_joint" type="revolute">
-    	<parent link="head_tilt_link" />
-    	<child link="upper_neck_link" />
-    	<origin xyz="0 0 0.013" rpy="0 0 0" />
+	<joint name="head_tilt_joint" type="revolute">
+    	<parent link="head_pan_link" />
+	<child link="head_tilt_link" />
+    	<origin xyz="0 0 0.044" rpy="0 0 0" />
     	<axis xyz="0 1 0" />
     	<limit lower="-1.57" upper="1.57" effort="10" velocity="3" />
       	<dynamics damping="0.0"/>
 	</joint>
- 	<joint name="upper_neck_joint" type="fixed">
-    	<parent link="upper_neck_link" />
+	<joint name="upper_neck_joint" type="fixed">
+    	<parent link="head_tilt_link" />
     	<child link="head_base_link" />
-    	<origin xyz="0 0 0.040" rpy="0 0 0" />
+    	<origin xyz="0 0 0.030" rpy="0 0 0" />
 	</joint>
 	<joint name="head_base_joint" type="fixed">
     	<parent link="head_base_link" />
     	<child link="head_post_link" />
-    	<origin xyz="0 0 0.016" rpy="0 0 0" />
+    	<origin xyz="0 0 0.022" rpy="0 0 0" />
 	</joint>
 	<joint name="head_joint" type="fixed">
     	<parent link="head_post_link" />
     	<child link="head_link" />
-    	<origin xyz="0 0 0.0235" rpy="0 0 0" />
+    	<origin xyz="0 0 0.012" rpy="0 0 0" />
 	</joint>
 	<joint name="left_eye_joint" type="fixed">
     	<parent link="head_link" />
     	<child link="left_eye_link" />
-    	<origin xyz="0.026 0.05 0" rpy="0 1.57 0" />
+    	<origin xyz="0.026 0.05 0.0175" rpy="0 1.57 0" />
 	</joint>
 	<joint name="right_eye_joint" type="fixed">
     	<parent link="head_link" />
     	<child link="right_eye_link" />
-    	<origin xyz="0.026 -0.05 0" rpy="0 1.57 0" />
-	</joint>
-	<!-- arm joints -->
-<!--        <joint name="finger_joint" type="fixed">
-	  <parent link="hand_link" />
-	  <child link="finger_link" />
-	  <origin xyz="0 0 -0.064" rpy="0 0 0" />
-        </joint>-->
+    	<origin xyz="0.026 -0.05 0.0175" rpy="0 1.57 0" />
+	</joint>
+	<!-- Arm Joints -->
 	<joint name="hand_joint" type="fixed">
 	  <parent link="wrist_roll_link" />
